Commit message: pip packaging things

File: iris_environments/assets/models/iiwa_description/urdf/iiwa14_spheres_collision.urdf (robot description, URDF)
Before this commit: robot iiwa14, 11 links, 10 joints
Links:
- link iiwa_link_0: geometry collision cylinder length=0.17 radius=0.139; visual mesh filename=package://iris_environments/models/iiwa_description/meshes/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
- link iiwa_link_1: geometry collision sphere radius=0.07959901601; visual mesh filename=package://iris_environments/models/iiwa_description/meshes/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
- link iiwa_link_2: geometry collision sphere radius=0.06602481863; collision sphere radius=0.07959901601
- link iiwa_link_3: geometry collision sphere radius=0.06062598796; collision sphere radius=0.06602481863
- link iiwa_link_4: geometry collision sphere radius=0.05993984276; collision sphere radius=0.06644602201
- link iiwa_link_5: geometry collision sphere radius=0.05281876964; collision sphere radius=0.06644602201
- link iiwa_link_6: geometry collision sphere radius=0.06341754633; visual mesh filename=package://iris_environments/models/iiwa_description/meshes/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
- link iiwa_link_7: geometry collision sphere radius=0.05285650291; visual mesh filename=package://iris_environments/models/iiwa_description/meshes/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
