Commit message: mycobot env for annan

File: iris_environments/assets/mycobot_description/urdf/mycobot/mycobot_with_gripper_parallel_obj.urdf (robot description, URDF)
Before this commit: robot firefighter, 15 links, 14 joints
Links:
- link g_base: geometry collision box size=0.152000 0.034000 0.111987; visual mesh filename=package://mycobot_description/urdf/mycobot/G_base.obj
- link gripper_base: geometry collision box size=0.060000 0.073525 0.055700; visual mesh filename=package://mycobot_description/urdf/mycobot/gripper_base.obj
- link gripper_left1: geometry collision box size=0.061259 0.028367 0.024333; visual mesh filename=package://mycobot_description/urdf/mycobot/gripper_left1.obj
- link gripper_left2: geometry collision box size=0.042015 0.022000 0.011000; visual mesh filename=package://mycobot_description/urdf/mycobot/gripper_left2.obj
- link gripper_left3: geometry collision box size=0.007000 0.042170 0.042139; visual mesh filename=package://mycobot_description/urdf/mycobot/gripper_left3.obj
- link gripper_right1: geometry collision box size=0.061259 0.028367 0.024333; visual mesh filename=package://mycobot_description/urdf/mycobot/gripper_right1.o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
- link gripper_right2: geometry collision box size=0.042015 0.022000 0.011000; visual mesh filename=package://mycobot_description/urdf/mycobot/gripper_right2.o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
- link gripper_right3: geometry collision box size=0.007000 0.037764 0.045797; visual mesh filename=package://mycobot_description/urdf/mycobot/gripper_right3.o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
- link joint1: geometry collision box size=0.092000 0.098794 0.075000; visual mesh filename=package://mycobot_description/urdf/mycobot/joint1.obj
- link joint2: geometry collision box size=0.062540 0.050000 0.089060; visual mesh filename=package://mycobot_description/urdf/mycobot/joint2.obj
- link joint3: geometry collision box size=0.057440 0.050000 0.158000; visual mesh filename=package://mycobot_description/urdf/mycobot/joint3.obj
- link joint4: geometry collision box size=0.059800 0.045200 0.138800; visual mesh filename=package://mycobot_description/urdf/mycobot/joint4.obj
- link joint5: geometry collision box size=0.040586 0.054786 0.058343; visual mesh filename=package://mycobot_description/urdf/mycobot/joint5.obj
- link joint6: geometry collision box size=0.040400 0.058700 0.059120; visual mesh filename=package://mycobot_description/urdf/mycobot/joint6.obj
- link joint6_flange: geometry collision box size=0.040400 0.040400 0.015700; visual mesh filename=package://mycobot_description/urdf/mycobot/joint7.obj
