Commit message: fixed 14dof env

File: iris_environments/assets_bimanual/models/iiwa_convex/iiwa14_convex_collision.urdf (robot description, URDF)
Before this commit: robot iiwa14, 11 links, 10 joints
Links:
- link iiwa_link_0: geometry collision mesh filename=package://bimanual/models/iiwa_convex/meshes/link_0_convex.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; visual mesh filename=package://iris_environments/models/iiwa_description/meshes/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
- link iiwa_link_1: geometry collision mesh filename=package://bimanual/models/iiwa_convex/meshes/link_1_convex.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; visual mesh filename=package://iris_environments/models/iiwa_description/meshes/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
- link iiwa_link_2: geometry collision mesh filename=package://bimanual/models/iiwa_convex/meshes/link_2_convex.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; visual mesh filename=package://iris_environments/models/iiwa_description/meshes/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
- link iiwa_link_3: geometry collision mesh filename=package://bimanual/models/iiwa_convex/meshes/link_3_convex.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; visual mesh filename=package://iris_environments/models/iiwa_description/meshes/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
- link iiwa_link_4: geometry collision mesh filename=package://bimanual/models/iiwa_convex/meshes/link_4_convex.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; visual mesh filename=package://iris_environments/models/iiwa_description/meshes/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
- link iiwa_link_5: geometry collision mesh filename=package://bimanual/models/iiwa_convex/meshes/link_5_convex.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; visual mesh filename=package://iris_environments/models/iiwa_description/meshes/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
- link iiwa_link_6: geometry collision mesh filename=package://bimanual/models/iiwa_convex/meshes/link_6_convex.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; visual mesh filename=package://iris_environments/models/iiwa_description/meshes/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
- link iiwa_link_7: geometry collision mesh filename=package://bimanual/models/iiwa_convex/meshes/link_7_convex.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; visual mesh filename=package://iris_environments/models/iiwa_description/meshes/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
