Commit message: fixed urdf conversion

File: iris_environments/assets/models/iiwa_description/iiwa7/iiwa7_with_box_collision.urdf (robot description, URDF)
Before this commit: robot iiwa7, 8 links, 7 joints
Joints:
- joint iiwa_joint_1: axis 0 0 1 -> 0.0 0.0 1.0; limit (none) -> lower=-2.96706 upper=2.96706 effort=300 velocity=10
- joint iiwa_joint_2: axis -0 1 0 -> -2.260097275516194e-27 6.123270170149069e-17 1.0; limit (none) -> lower=-2.0944 upper=2.0944 effort=300 velocity=10
- joint iiwa_joint_3: axis 0 0 1 -> -1.61558713389832e-27 3.6732051034078064e-06 0.9999999999932537; limit (none) -> lower=-2.96706 upper=2.96706 effort=300 velocity=10; origin xyz=-4.434786682550889e-28 0.18399999999875866 -6.758697390157694e-07 rpy=1.5708 2.653589793337943e-06 -3.1415926535800462 -> xyz=-4.434786682550889e-28 0.18399999999875866 -6.758697390157694e-07 rpy=1.5708 2.6535897933379433e-06 -3.1415926535800462
- joint iiwa_joint_4: axis 0 -1 0 -> 0.0 -6.123270170149069e-17 -1.0; limit (none) -> lower=-2.0944 upper=2.0944 effort=300 velocity=10
- joint iiwa_joint_5: axis 0 0 1 -> -2.6535897933348283e-06 3.6732051032853415e-06 -0.999999999989733; limit (none) -> lower=-2.96706 upper=2.96706 effort=300 velocity=10
- joint iiwa_joint_6: axis -0 1 -0 -> 9.747179571131627e-12 7.3464102066918875e-06 0.9999999999730153; limit (none) -> lower=-2.0944 upper=2.0944 effort=300 velocity=10
- joint iiwa_joint_7: axis 0 0 1 -> -1.61558713389832e-27 3.6732051034078064e-06 0.9999999999932537; limit (none) -> lower=-3.05433 upper=3.05433 effort=300 velocity=10; origin xyz=-1.9710163033559505e-27 0.08049999999945712 -2.956930108193996e-07 rpy=1.5708 2.653589793337943e-06 -3.1415926535800462 -> xyz=-1.9710163033559505e-27 0.08049999999945712 -2.956930108193996e-07 rpy=1.5708 2.6535897933379433e-06 -3.1415926535800462

Commit message: triangle example

File: iris_environments/assets/models/iiwa_description/iiwa7/iiwa7_with_box_collision.urdf (robot description, URDF)
Before this commit: robot iiwa7, 8 links, 7 joints
Joints:
- joint iiwa_joint_2: axis -2.260097275516194e-27 6.123270170149069e-17 1.0 -> -2.65358979335273e-06 3.6732051033336423e-06 0.9999999999897331
- joint iiwa_joint_3: axis -1.61558713389832e-27 3.6732051034078064e-06 0.9999999999932537 -> 2.6535897933254864e-06 7.041525858790415e-12 0.9999999999964793
- joint iiwa_joint_4: axis 0.0 -6.123270170149069e-17 -1.0 -> 0.0 3.6732051033465748e-06 0.9999999999932538
- joint iiwa_joint_5: axis -2.6535897933348283e-06 3.6732051032853415e-06 -0.999999999989733 -> 2.6535897933348288e-06 1.293243726632807e-17 0.9999999999964793
- joint iiwa_joint_6: axis 9.747179571131627e-12 7.3464102066918875e-06 0.9999999999730153 -> -9.747179570748406e-12 3.6732051033336423e-06 0.9999999999932538
- joint iiwa_joint_7: axis -1.61558713389832e-27 3.6732051034078064e-06 0.9999999999932537 -> 2.6535897933254864e-06 7.041525858790415e-12 0.9999999999964793

File: iris_environments/assets/models/shelves/shelves.urdf (robot description, URDF)
Before this commit: robot shelves, 2 links, 1 joints
Links:
- link shelves_body: geometry collision box size=0.3 0.016 0.783; collision box size=0.3 0.016 0.783
Joints:
- joint top_and_bottom_shelves_body: origin (none) -> xyz=0.0 0.0 0.0 rpy=0.0 -0.0 0.0
